File: UINIO-MCU-STM32F401CCU6.kicad_sch (KiCad schematic)
At the start: 37 parts, among them J1 Conn_01x24_Pin, J2 Conn_01x24_Pin, J3 Conn_01x04_Pin, SW1 BOOT1, SW2 NRST, SW3 BOOT0, U1 ME6211C33M5G-N, U3 STM32F401CCU6, Y1 32.768KHz, Y2 8MHz

Commit message: Release UINIO-MCU-STM32F401CCU6 version 3.1.0.
Connections:
- net GND: now also L1.1; no longer U3.8 (VSSA)
- net VDD_3.3V: now also U3.9 (VDDA); no longer L1.1
- net at L1.2: now also U3.8 (VSSA); no longer U3.9 (VDDA)
Other:
- moved on the sheet: L1
Changed lines of the file:
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@@
   (title_block
     (title "UINIO-MCU-STM32F401CCU6")
-    (date "2024-02-06")
-    (rev "Version 3.0.0")
+    (date "2024-04-12")
+    (rev "Version 3.1.0")
     (company "UinIO.com 电子技术工作室")
   )
@@
     (stroke (width 0) (type default))
   )
+  (wire (pts (xy 238.76 113.03) (xy 247.65 113.03))
+    (stroke (width 0) (type default))
+  )
   (wire (pts (xy 247.65 99.06) (xy 250.19 99.06))
     (stroke (width 0) (type default))
@@
     (stroke (width 0) (type default))
   )
-  (wire (pts (xy 236.22 118.11) (xy 255.27 118.11))
-    (stroke (width 0) (type default))
-  )
   (wire (pts (xy 33.02 50.8) (xy 34.29 50.8))
+    (stroke (width 0) (type default))
+  )
+  (wire (pts (xy 214.63 118.11) (xy 255.27 118.11))
     (stroke (width 0) (type default))
   )
@@
     (stroke (width 0) (type default))
   )
-  (wire (pts (xy 217.17 113.03) (xy 241.3 113.03))
+  (wire (pts (xy 217.17 113.03) (xy 231.14 113.03))
     (stroke (width 0) (type default))
   )
@@
   )
   (wire (pts (xy 33.02 78.74) (xy 34.29 78.74))
-    (stroke (width 0) (type default))
-  )
-  (wire (pts (xy 228.6 118.11) (xy 214.63 118.11))
     (stroke (width 0) (type default))
   )
@@
     )
   )
-  (symbol (lib_id "power:GND") (at 241.3 113.03 90) (mirror x) (unit 1)
-    (in_bom yes) (on_board yes) (dnp no)
-    (property "Reference" "#PWR022" (at 247.65 113.03 0)
-      (effects (font (size 1.27 1.27)) hide)
-    )
-    (property "Value" "GND" (at 244.475 113.03 90)
+  (symbol (lib_id "power:GND") (at 247.65 113.03 90) (mirror x) (unit 1)
+    (in_bom yes) (on_board yes) (dnp no)
+    (property "Reference" "#PWR022" (at 254 113.03 0)
+      (effects (font (size 1.27 1.27)) hide)
+    )
+    (property "Value" "GND" (at 250.825 113.03 90)
       (effects (font (size 1.27 1.27)) (justify right))
     )
-    (property "Footprint" "" (at 241.3 113.03 0)
-      (effects (font (size 1.27 1.27)) hide)
-    )
-    (property "Datasheet" "" (at 241.3 113.03 0)
+    (property "Footprint" "" (at 247.65 113.03 0)
+      (effects (font (size 1.27 1.27)) hide)
+    )
+    (property "Datasheet" "" (at 247.65 113.03 0)
       (effects (font (size 1.27 1.27)) hide)
     )
@@
     )
   )
-  (symbol (lib_id "Device:L") (at 232.41 118.11 270) (mirror x) (unit 1)
-    (in_bom yes) (on_board yes) (dnp no)
-    (property "Reference" "L1" (at 229.87 119.38 90)
+  (symbol (lib_id "Device:L") (at 234.95 113.03 270) (mirror x) (unit 1)
+    (in_bom yes) (on_board yes) (dnp no)
+    (property "Reference" "L1" (at 232.41 114.3 90)
       (effects (font (size 1.27 1.27)) (justify right))
     )
-    (property "Value" "1KΩ 100Mhz" (at 243.84 119.38 90)
+    (property "Value" "1KΩ 100Mhz" (at 246.38 114.3 90)
       (effects (font (size 1.27 1.27)) (justify right))
     )
-    (property "Footprint" "Inductor_SMD:L_0603_1608Metric" (at 232.41 118.11 0)
-      (effects (font (size 1.27 1.27)) hide)
-    )
-    (property "Datasheet" "~" (at 232.41 118.11 0)
-      (effects (font (size 1.27 1.27)) hide)
-    )
+    (property "Footprint" "Inductor_SMD:L_0603_1608Metric" (at 234.95 113.03 0)
+      (effects (font (size 1.27 1.27)) hide)
+    )
+    (property "Datasheet" "~" (at 234.95 113.03 0)
+      (effects (font (size 1.27 1.27)) hide)
+    )

Commit message: Release UINIO-MCU-STM32F401CCU6 version 3.2.0.
Connections:
- net PA11 renamed USB_PA-
- net PA12 renamed USB_PA+
Changed lines of the file:
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@@
   (title_block
     (title "UINIO-MCU-STM32F401CCU6")
-    (date "2024-04-12")
-    (rev "Version 3.1.0")
+    (date "2024-04-13")
+    (rev "Version 3.2.0")
     (company "UinIO.com 电子技术工作室")
   )
@@
     (effects (font (size 1.27 1.27)) (justify right bottom))
   )
-  (label "PA11" (at 129.54 66.04 180) (fields_autoplaced)
+  (label "~PA11" (at 129.54 66.04 180) (fields_autoplaced)
     (effects (font (size 1.27 1.27)) (justify right bottom))
   )
@@
     (effects (font (size 1.27 1.27)) (justify left bottom))
   )
+  (label "USB_PA+" (at 110.49 63.5 0) (fields_autoplaced)
+    (effects (font (size 1.27 1.27)) (justify left bottom))
+  )
   (label "PB8" (at 49.53 63.5 0) (fields_autoplaced)
     (effects (font (size 1.27 1.27)) (justify left bottom))
@@
     (effects (font (size 1.27 1.27)) (justify right bottom))
   )
-  (label "PA12" (at 33.02 45.72 180) (fields_autoplaced)
+  (label "~PA12" (at 33.02 45.72 180) (fields_autoplaced)
     (effects (font (size 1.27 1.27)) (justify right bottom))
   )
@@
     (effects (font (size 1.27 1.27)) (justify left bottom))
   )
+  (label "USB_PA-" (at 110.49 66.04 0) (fields_autoplaced)
+    (effects (font (size 1.27 1.27)) (justify left bottom))
+  )
   (label "PA14{slash}SWCLK" (at 49.53 43.18 0) (fields_autoplaced)
     (effects (font (size 1.27 1.27)) (justify left bottom))
@@
     (effects (font (size 1.27 1.27)) (justify right bottom))
   )
-  (label "PA11" (at 33.02 48.26 180) (fields_autoplaced)
+  (label "~PA11" (at 33.02 48.26 180) (fields_autoplaced)
     (effects (font (size 1.27 1.27)) (justify right bottom))
   )
@@
     (effects (font (size 1.27 1.27)) (justify left bottom))
   )
-  (label "PA12" (at 129.54 63.5 180) (fields_autoplaced)
-    (effects (font (size 1.27 1.27)) (justify right bottom))
-  )
+  (label "~PA12" (at 129.54 63.5 180) (fields_autoplaced)
+    (effects (font (size 1.27 1.27)) (justify right bottom))
+  )
