File: UINIO-MCU-STM32F401CCU6.kicad_pcb (KiCad board)
At the start: 2 copper layers, 68.4 x 20.3 mm, 41 parts, among them J1 Conn_01x24_Pin, J2 Conn_01x24_Pin, J3 Conn_01x04_Pin, SW1 BOOT1, SW2 NRST, SW3 BOOT0, U1 ME6211C33M5G-N, U3 STM32F401CCU6, Y1 32.768KHz, Y2 8MHz

Commit message: Release UINIO-MCU-STM32F401CCU6 version 3.1.0.
Parts:
- moved C12 0.32 mm to (161.5, 95.7)
- moved C8 0.32 mm to (161.5, 100.0)
- moved Y2 0.32 mm to (160.3, 97.9)
- moved C10 0.32 mm to (159.9, 103.8)
- moved C11 0.32 mm to (159.9, 102.0)
- moved Y1 0.32 mm to (161.4, 102.9)
Connections:
- L1 pad 1: /VDD_3.3V -> GND
- L1 pad 2: Net-(U3-VDDA) -> Net-(U3-VSSA)
- U3 pad 8: GND -> Net-(U3-VSSA)
- U3 pad 9: Net-(U3-VDDA) -> /VDD_3.3V
Routing:
- net GND: track 118.2 -> 94.6 mm, vias 46 -> 51
- net Net-(U3-VSSA): track 0.00 -> 21.1 mm
- net Net-(U3-VDDA): track 12.7 -> 0.00 mm, vias 2 -> 0
- net /PA12: track 35.9 -> 28.5 mm
- net /VDD_3.3V: track 167.3 -> 173.9 mm, vias 3 -> 5
- net Net-(U3-PD0_OSC_IN): track 10.1 -> 11.6 mm
- net Net-(U3-PD1_OSC_OUT): track 13.2 -> 14.6 mm
- net Net-(U3-PC15_OSC32_OUT): track 9.87 -> 11.0 mm
- net /NRST: track 40.8 -> 41.9 mm
Other:
- board text added: "Version 3.1.0"
- board text removed: "Version 3.0.0"

Commit message: Release UINIO-MCU-STM32F401CCU6 version 3.2.0.
Parts:
- moved R12 0.52 mm to (134.7, 100.5), turned to 0 degrees
Connections:
- net /PA11 renamed /USB_PA-
- net /PA12 renamed /USB_PA+
Routing:
- net GND: track 94.6 -> 105.2 mm, vias 51 -> 60
- net /USB_PA-: track 23.8 -> 26.3 mm, vias 0 -> 1
- net /VDD_3.3V: track 173.9 -> 175.5 mm
- net /USB_PA+: track 28.5 -> 29.3 mm
Other:
- board text added: "Version 3.2.0"
- board text removed: "Version 3.1.0"

Commit message: Release UINIO-MCU-STM32F401CCU6 version 3.2.0.
Routing:
- net GND: track 105.2 -> 104.2 mm, vias 60 -> 67
Changed lines of the file:
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@@
   (segment (start 160.13213 105.06213) (end 159.87094 104.80094) (width 0.3) (layer "F.Cu") (net 1))
   (segment (start 156.75 105.87) (end 156.43 105.55) (width 0.5) (layer "F.Cu") (net 1))
-  (segment (start 135.45 94.86) (end 132.698156 97.611844) (width 0.3) (layer "F.Cu") (net 1))
   (segment (start 162.80906 100.01213) (end 161.65906 100.01213) (width 0.3) (layer "F.Cu") (net 1))
   (segment (start 144.43 97.92) (end 145.264594 97.92) (width 0.3) (layer "F.Cu") (net 1))
@@
   (segment (start 162.80906 100.69213) (end 162.80906 100.01213) (width 0.3) (layer "F.Cu") (net 1))
   (segment (start 151.66 105.56) (end 152.78 105.56) (width 0.6) (layer "F.Cu") (net 1))
-  (segment (start 135.45 94.82) (end 135.45 94.86) (width 0.3) (layer "F.Cu") (net 1))
   (segment (start 119.19806 95.51713) (end 119.19806 104.16713) (width 0.5) (layer "F.Cu") (net 1))
   (segment (start 145.264594 97.92) (end 146.203196 98.858602) (width 0.3) (layer "F.Cu") (net 1))
@@
   (segment (start 156.43 105.55) (end 152.81 105.55) (width 0.5) (layer "F.Cu") (net 1))
   (segment (start 124.15906 96.64213) (end 123.39806 95.88113) (width 0.5) (layer "F.Cu") (net 1))
+  (segment (start 134.84 96.88) (end 134.85 96.87) (width 0.2) (layer "F.Cu") (net 1))
   (segment (start 123.39806 95.51713) (end 119.19806 95.51713) (width 0.5) (layer "F.Cu") (net 1))
   (segment (start 162.80906 100.79213) (end 162.80906 100.69213) (width 0.3) (layer "F.Cu") (net 1))
   (segment (start 150.62906 107.31) (end 151.57 107.31) (width 0.3) (layer "F.Cu") (net 1))
   (segment (start 131.08156 95.16) (end 126.65 95.16) (width 0.5) (layer "F.Cu") (net 1))
+  (via (at 134.85 96.87) (size 0.5) (drill 0.3) (layers "F.Cu" "B.Cu") (free) (net 1))
   (via (at 180.92333 99.86) (size 0.5) (drill 0.3) (layers "F.Cu" "B.Cu") (free) (net 1))
   (via (at 156.75 105.87) (size 0.7) (drill 0.3) (layers "F.Cu" "B.Cu") (free) (net 1))
@@
   (via (at 136.13 104.91) (size 0.5) (drill 0.3) (layers "F.Cu" "B.Cu") (free) (net 1))
   (via (at 175.84 99.86) (size 0.5) (drill 0.3) (layers "F.Cu" "B.Cu") (free) (net 1))
+  (via (at 134.91 94.7) (size 0.5) (drill 0.3) (layers "F.Cu" "B.Cu") (free) (net 1))
   (via (at 163.68 95.44) (size 0.7) (drill 0.3) (layers "F.Cu" "B.Cu") (net 1))
   (via (at 150.26906 99.742485) (size 0.5) (drill 0.3) (layers "F.Cu" "B.Cu") (net 1))
@@
   (via (at 177.46906 92.99213) (size 0.5) (drill 0.3) (layers "F.Cu" "B.Cu") (free) (net 1))
   (via (at 149.53 92.56) (size 0.5) (drill 0.3) (layers "F.Cu" "B.Cu") (free) (net 1))
+  (via (at 133.72 97.77) (size 0.5) (drill 0.3) (layers "F.Cu" "B.Cu") (free) (net 1))
   (via (at 179.906664 99.86) (size 0.5) (drill 0.3) (layers "F.Cu" "B.Cu") (free) (net 1))
+  (via (at 134.26 94.04) (size 0.5) (drill 0.3) (layers "F.Cu" "B.Cu") (free) (net 1))
   (via (at 180.82 105.32) (size 0.5) (drill 0.3) (layers "F.Cu" "B.Cu") (free) (net 1))
   (via (at 152.81 105.55) (size 0.7) (drill 0.3) (layers "F.Cu" "B.Cu") (net 1))
@@
   (via (at 169.79656 92.99213) (size 0.5) (drill 0.3) (layers "F.Cu" "B.Cu") (free) (net 1))
   (via (at 128.67 98.35) (size 0.5) (drill 0.3) (layers "F.Cu" "B.Cu") (free) (net 1))
+  (via (at 137.87 95.38) (size 0.5) (drill 0.3) (layers "F.Cu" "B.Cu") (free) (net 1))
   (via (at 169.26 104.78) (size 0.5) (drill 0.3) (layers "F.Cu" "B.Cu") (free) (net 1))
   (via (at 172.35406 92.99213) (size 0.5) (drill 0.3) (layers "F.Cu" "B.Cu") (free) (net 1))
   (via (at 166.38 104.78) (size 0.5) (drill 0.3) (layers "F.Cu" "B.Cu") (free) (net 1))
+  (via (at 133.61 93.41) (size 0.5) (drill 0.3) (layers "F.Cu" "B.Cu") (free) (net 1))
   (via (at 149.26906 100.742485) (size 0.5) (drill 0.3) (layers "F.Cu" "B.Cu") (net 1))
   (via (at 172.48 101.67) (size 0.7) (drill 0.3) (layers "F.Cu" "B.Cu") (free) (net 1))
@@
   (via (at 157.93 107.05) (size 0.7) (drill 0.3) (layers "F.Cu" "B.Cu") (net 1))
   (via (at 162.79906 105.06213) (size 0.7) (drill 0.3) (layers "F.Cu" "B.Cu") (net 1))
-  (via (at 135.45 94.82) (size 0.7) (drill 0.3) (layers "F.Cu" "B.Cu") (net 1))
+  (via (at 139.93 95.38) (size 0.5) (drill 0.3) (layers "F.Cu" "B.Cu") (free) (net 1))
+  (via (at 138.9 95.38) (size 0.5) (drill 0.3) (layers "F.Cu" "B.Cu") (free) (net 1))
   (via (at 151.26906 100.742485) (size 0.5) (drill 0.3) (layers "F.Cu" "B.Cu") (net 1))
   (via (at 160.16 107.05) (size 0.7) (drill 0.3) (layers "F.Cu" "B.Cu") (net 1))
@@
   (segment (start 137.72 97.77) (end 134.87 97.77) (width 0.5) (layer "B.Cu") (net 1))
   (segment (start 152.79 105.55) (end 152.81 105.57) (width 0.3) (layer "B.Cu") (net 1))
+  (segment (start 134.85 96.87) (end 137.72 96.87) (width 0.5) (layer "B.Cu") (net 1))
   (segment (start 164.1 95.86) (end 167.78163 95.86) (width 0.3) (layer "B.Cu") (net 1))
   (segment (start 167.78163 95.86) (end 168.16 95.48163) (width 0.3) (layer "B.Cu") (net 1))
@@
         (xy 138.16 96.9)
         (xy 138.16 99.93)
-        (xy 138.16 99.93)
         (xy 134.34 99.93)
         (xy 134.34 96.9)
-        (xy 134.34 96.9)
       )

Commit message: Release UINIO-MCU-STM32F401CCU6 version 3.2.0.
Parts:
- moved R1 2.29 mm to (134.2, 95.7), turned to -90 degrees
- moved R11 0.54 mm to (132.2, 97.1)
- moved R12 0.47 mm to (134.7, 101.0)
Routing:
- net GND: track 104.2 -> 103.1 mm, vias 67 -> 70
- net /VDD_3.3V: track 175.5 -> 174.8 mm
